Commit message: fix(calib): add missing origin elements in inertial, collision, and visual sections

File: denso_robot_descriptions/tools/calib/urdf/calib.xacro (robot description, xacro)
@@ -4,8 +4,10 @@
     <link name="${namespace}calib_link">
 		<inertial>
+			<origin rpy="${rpy}" xyz="${xyz}"/>
 			<mass value="0.1"/>
 			<inertia ixx="0.001" ixy="0" ixz="0" iyy="0.001" iyz="0" izz="0.001"/>
 		</inertial>
 		<collision>
+			<origin rpy="${rpy}" xyz="${xyz}"/>
 			<geometry>
 				<mesh filename="file:///$(find denso_robot_descriptions)/tools/calib/meshes/apex_v3_1.stl" scale="0.001 0.001 0.001"/>
@@ -13,4 +15,5 @@
 		</collision>
 		<visual>
+			<origin rpy="${rpy}" xyz="${xyz}"/>
 			<geometry>
 				<mesh filename="file:///$(find denso_robot_descriptions)/tools/calib/meshes/apex_v3_1.stl" scale="0.001 0.001 0.001"/>
