Commit message: feat(calibration): add calibration tool support with configurable parameters

File: denso_robot_descriptions/robots/vs050/urdf/denso_robot_macro.xacro (robot description, xacro)
@@ -17,4 +17,7 @@
     sim:=false
     basic_camera:=false
+    calib_tool:=false
+    calib_xyz:='0 0 0.01'
+    calib_rpy:='0 0 0'
     ip_address
     send_format
@@ -52,4 +55,7 @@
       <xacro:include filename="$(find denso_robot_descriptions)/tools/basic_camera/urdf/basic_camera.xacro" />
     </xacro:if>
+    <xacro:if value="$(arg calib_tool)">
+      <xacro:include filename="$(find denso_robot_descriptions)/tools/calib/urdf/calib.xacro" />
+    </xacro:if>
     <!-- ros2 control instance -->
     <xacro:denso_robot_ros2_control
@@ -82,4 +88,11 @@
       <xacro:basic_camera namespace="${namespace}" end_effector="J6" />
     </xacro:if>
+    <xacro:if value="$(arg calib_tool)">
+      <xacro:calib
+        namespace="${namespace}"
+        end_effector="J6"
+        xyz="$(arg calib_xyz)"
+        rpy="$(arg calib_rpy)" />
+    </xacro:if>
   </xacro:macro>
 </robot>

File: denso_robot_descriptions/urdf/denso_robot.urdf.xacro (robot description, xacro)
@@ -12,4 +12,7 @@
    <xacro:arg name="sim" default="false" />
    <xacro:arg name="basic_camera" default="false" />
+  <xacro:arg name="calib_tool" default="false" />
+  <xacro:arg name="calib_xyz" default="0 0 0.01" />
+  <xacro:arg name="calib_rpy" default="0 0 0" />
    <xacro:arg name="ip_address" default="192.168.0.1" />
    <xacro:arg name="send_format" default="288" />
@@ -27,4 +30,7 @@
      sim="$(arg sim)"
      basic_camera="$(arg basic_camera)"
+    calib_tool="$(arg calib_tool)"
+    calib_xyz="$(arg calib_xyz)"
+    calib_rpy="$(arg calib_rpy)"
      ip_address="$(arg ip_address)"
      verbose="$(arg verbose)"

File: denso_robot_moveit_config/robots/vs050/srdf/denso_robot_macro.srdf.xacro (robot description, xacro)
@@ -5,5 +5,5 @@
     A URDF file must exist for this robot as well, where the joints and the links that are referenced are defined
 -->
-  <xacro:macro name="denso_robot_srdf" params="namespace">
+	<xacro:macro name="denso_robot_srdf" params="namespace calib_tool:=false">
     <!--GROUPS - Representation of a set of joints and links. This can be useful for specifying DOF to plan for, defining arms, end effectors, etc-->
     <!--LINKS - When a link is specified, the parent joint of that link (if it exists) is automatically included-->
@@ -32,4 +32,8 @@
 	<disable_collisions link1="${namespace}J3" link2="${namespace}J5" reason="Never"/>
 	<disable_collisions link1="${namespace}J4" link2="${namespace}J5" reason="Adjacent"/>
+    <xacro:if value="${calib_tool}">
+	  <disable_collisions link1="${namespace}J6" link2="${namespace}calib_link" reason="Adjacent"/>
+	  <disable_collisions link1="${namespace}J5" link2="${namespace}calib_link" reason="Never"/>
+    </xacro:if>
   </xacro:macro>
 </robot>

File: denso_robot_moveit_config/srdf/denso_robot.srdf.xacro (robot description, xacro)
@@ -5,5 +5,6 @@
   <!-- parameters -->
   <xacro:arg name="namespace" default="" />
+  <xacro:arg name="calib_tool" default="false" />
   <xacro:include filename="$(find denso_robot_moveit_config)/robots/$(arg model)/srdf/denso_robot_macro.srdf.xacro"/>
-  <xacro:denso_robot_srdf namespace="$(arg namespace)"/>
+  <xacro:denso_robot_srdf namespace="$(arg namespace)" calib_tool="$(arg calib_tool)"/>
 </robot>

Commit message: feat(calib): add mesh offset parameters for calibration tool in launch files and xacro macros

File: denso_robot_descriptions/robots/vs050/urdf/denso_robot_macro.xacro (robot description, xacro)
@@ -20,4 +20,6 @@
     calib_xyz:='0 0 0.01'
     calib_rpy:='0 0 0'
+    calib_mesh_xyz:='0.01 0.004 0.946'
+    calib_mesh_rpy:='0 0 0'
     ip_address
     send_format
@@ -93,5 +95,7 @@
         end_effector="J6"
         xyz="$(arg calib_xyz)"
-        rpy="$(arg calib_rpy)" />
+        rpy="$(arg calib_rpy)"
+        mesh_xyz="$(arg calib_mesh_xyz)"
+        mesh_rpy="$(arg calib_mesh_rpy)" />
     </xacro:if>
   </xacro:macro>

File: denso_robot_descriptions/tools/calib/urdf/calib.xacro (robot description, xacro)
@@ -1,5 +1,5 @@
 <?xml version='1.0' encoding='UTF-8'?>
 <robot xmlns:xacro="http://www.ros.org/wiki/xacro">
-    <xacro:macro name="calib" params="namespace end_effector xyz rpy">
+    <xacro:macro name="calib" params="namespace end_effector xyz rpy mesh_xyz:='0.01 0.004 0.946' mesh_rpy:='0 0 0'">
     <link name="${namespace}calib_link">
 		<inertial>
@@ -9,5 +9,5 @@
 		</inertial>
 		<collision>
-			<origin rpy="${rpy}" xyz="${xyz}"/>
+			<origin rpy="${mesh_rpy}" xyz="${mesh_xyz}"/>
 			<geometry>
 				<mesh filename="file:///$(find denso_robot_descriptions)/tools/calib/meshes/apex_v3_1.stl" scale="0.001 0.001 0.001"/>
@@ -15,5 +15,5 @@
 		</collision>
 		<visual>
-			<origin rpy="${rpy}" xyz="${xyz}"/>
+			<origin rpy="${mesh_rpy}" xyz="${mesh_xyz}"/>
 			<geometry>
 				<mesh filename="file:///$(find denso_robot_descriptions)/tools/calib/meshes/apex_v3_1.stl" scale="0.001 0.001 0.001"/>

File: denso_robot_descriptions/urdf/denso_robot.urdf.xacro (robot description, xacro)
@@ -15,4 +15,6 @@
   <xacro:arg name="calib_xyz" default="0 0 0.01" />
   <xacro:arg name="calib_rpy" default="0 0 0" />
+  <xacro:arg name="calib_mesh_xyz" default="0.01 0.004 0.946" />
+  <xacro:arg name="calib_mesh_rpy" default="0 0 0" />
    <xacro:arg name="ip_address" default="192.168.0.1" />
    <xacro:arg name="send_format" default="288" />
@@ -33,4 +35,6 @@
     calib_xyz="$(arg calib_xyz)"
     calib_rpy="$(arg calib_rpy)"
+    calib_mesh_xyz="$(arg calib_mesh_xyz)"
+    calib_mesh_rpy="$(arg calib_mesh_rpy)"
      ip_address="$(arg ip_address)"
      verbose="$(arg verbose)"

Commit message: [REFACTOR]: cleaner tool spawning using the new .dae file

File: denso_robot_descriptions/robots/vs050/urdf/denso_robot_macro.xacro (robot description, xacro)
@@ -20,5 +20,5 @@
     calib_xyz:='0 0 0.01'
     calib_rpy:='0 0 0'
-    calib_mesh_xyz:='0.01 0.004 0.946'
+    calib_mesh_xyz:='0 0 0'
     calib_mesh_rpy:='0 0 0'
     ip_address
@@ -58,5 +58,5 @@
     </xacro:if>
     <xacro:if value="$(arg calib_tool)">
-      <xacro:include filename="$(find denso_robot_descriptions)/tools/calib/urdf/calib.xacro" />
+      <xacro:include filename="$(find denso_robot_descriptions)/tools/calibration_tool/urdf/calib.xacro" />
     </xacro:if>
     <!-- ros2 control instance -->

File: denso_robot_descriptions/tools/calibration_tool/urdf/calib.xacro (robot description, xacro)
@@ -1,5 +1,5 @@
 <?xml version='1.0' encoding='UTF-8'?>
 <robot xmlns:xacro="http://www.ros.org/wiki/xacro">
-    <xacro:macro name="calib" params="namespace end_effector xyz rpy mesh_xyz:='0.01 0.004 0.946' mesh_rpy:='0 0 0'">
+	<xacro:macro name="calib" params="namespace end_effector xyz rpy mesh_xyz:='0 0 0' mesh_rpy:='0 0 0'">
     <link name="${namespace}calib_link">
 		<inertial>
@@ -11,5 +11,5 @@
 			<origin rpy="${mesh_rpy}" xyz="${mesh_xyz}"/>
 			<geometry>
-				<mesh filename="file:///$(find denso_robot_descriptions)/tools/calib/meshes/apex_v3_1.stl" scale="0.001 0.001 0.001"/>
+				<mesh filename="file:///$(find denso_robot_descriptions)/tools/calibration_tool/meshes/calibration_tool.dae" scale="0.001 0.001 0.001"/>
 			</geometry>
 		</collision>
@@ -17,5 +17,5 @@
 			<origin rpy="${mesh_rpy}" xyz="${mesh_xyz}"/>
 			<geometry>
-				<mesh filename="file:///$(find denso_robot_descriptions)/tools/calib/meshes/apex_v3_1.stl" scale="0.001 0.001 0.001"/>
+				<mesh filename="file:///$(find denso_robot_descriptions)/tools/calibration_tool/meshes/calibration_tool.dae" scale="0.001 0.001 0.001"/>
 			</geometry>
 		</visual>

File: denso_robot_descriptions/urdf/denso_robot.urdf.xacro (robot description, xacro)
@@ -15,5 +15,5 @@
   <xacro:arg name="calib_xyz" default="0 0 0.01" />
   <xacro:arg name="calib_rpy" default="0 0 0" />
-  <xacro:arg name="calib_mesh_xyz" default="0.01 0.004 0.946" />
+  <xacro:arg name="calib_mesh_xyz" default="0 0 0" />
   <xacro:arg name="calib_mesh_rpy" default="0 0 0" />
    <xacro:arg name="ip_address" default="192.168.0.1" />
