Commit message: feat: add camera to dual Denso robot launch configuration

File: denso_robot_descriptions/robots/vs050/urdf/denso_robot_macro.xacro (robot description, xacro)
@@ -61,5 +61,5 @@
     <!-- The line with tag xacro:tool passes the parameters defined in your tool's xacro file -->
     <!-- (see basic_camera.xacro as an example implementation) -->
-    <xacro:if value="$(arg basic_camera)">
+    <xacro:if value="${basic_camera}">
       <xacro:include filename="$(find denso_robot_descriptions)/tools/basic_camera/urdf/basic_camera.xacro" />
     </xacro:if>
@@ -97,5 +97,5 @@
       <xacro:insert_block name="origin" />
     </xacro:denso_robot_arm_kinematics>
-    <xacro:if value="$(arg basic_camera)">
+    <xacro:if value="${basic_camera}">
       <xacro:basic_camera namespace="${namespace}" end_effector="J6" />
     </xacro:if>

File: denso_robot_descriptions/robots/vs060/urdf/denso_robot_macro.xacro (robot description, xacro)
@@ -61,5 +61,5 @@
     <!-- The line with tag xacro:tool passes the parameters defined in your tool's xacro file -->
     <!-- (see basic_camera.xacro as an example implementation) -->
-    <xacro:if value="$(arg basic_camera)">
+    <xacro:if value="${basic_camera}">
       <xacro:include filename="$(find denso_robot_descriptions)/tools/basic_camera/urdf/basic_camera.xacro" />
     </xacro:if>
@@ -97,5 +97,5 @@
       <xacro:insert_block name="origin" />
     </xacro:denso_robot_arm_kinematics>
-    <xacro:if value="$(arg basic_camera)">
+    <xacro:if value="${basic_camera}">
       <xacro:basic_camera namespace="${namespace}" end_effector="J6" />
     </xacro:if>

File: denso_robot_descriptions/tools/basic_camera/urdf/basic_camera.xacro (robot description, xacro)
@@ -5,4 +5,10 @@
     <!-- if your tool has meshes, define the path to it in geometry tag. -->
     <!-- see the vs050 robot urdf implementation as an example. -->
+    <material name="${namespace}basic_camera_body_material">
+      <color rgba="0.05 0.16 0.30 1.0"/>
+    </material>
+    <material name="${namespace}basic_camera_view_axis_material">
+      <color rgba="0.0 0.75 1.0 0.55"/>
+    </material>
     <link name="${namespace}basic_camera_link">
 		<inertial>
@@ -12,13 +18,28 @@
 		<collision>
 			<geometry>
-				<box size="0.01 0.01 0.01"/>
+				<box size="0.035 0.03 0.025"/>
 			</geometry>
 		</collision>
 		<visual>
 			<geometry>
-				<box size="0.01 0.01 0.01"/>
+				<box size="0.035 0.03 0.025"/>
 			</geometry>
+      <material name="${namespace}basic_camera_body_material"/>
 		</visual>
 	</link>
+  <link name="${namespace}basic_camera_view_axis">
+    <visual>
+      <origin rpy="0 1.57079632679 0" xyz="0.13 0 0"/>
+      <geometry>
+        <cylinder length="0.26" radius="0.003"/>
+      </geometry>
+      <material name="${namespace}basic_camera_view_axis_material"/>
+    </visual>
+  </link>
+  <joint name="${namespace}basic_camera_view_axis_joint" type="fixed">
+    <parent link="${namespace}basic_camera_link"/>
+    <child link="${namespace}basic_camera_view_axis"/>
+    <origin rpy="0 0 0" xyz="0 0 0"/>
+  </joint>
 	<joint name="${namespace}basic_camera_joint" type="fixed">
         <!-- here you define where your tool will connect. In this case, it's at joint 6. -->

File: denso_robot_descriptions/urdf/dual_denso_robot.urdf.xacro (robot description, xacro)
@@ -10,5 +10,6 @@
    <xacro:arg name="verbose" default="false" />
    <xacro:arg name="sim" default="false" />
-   <xacro:arg name="basic_camera" default="false" />
+   <xacro:arg name="left_basic_camera" default="true" />
+   <xacro:arg name="right_basic_camera" default="false" />
    <xacro:arg name="left_ip_address" default="192.168.0.1" />
    <xacro:arg name="right_ip_address" default="192.168.0.2" />
@@ -17,5 +18,5 @@
    <xacro:arg name="calib_tool" default="false" />
    <xacro:arg name="left_cellphone_holder" default="false" />
-   <xacro:arg name="right_cellphone_holder" default="false" />
+   <xacro:arg name="right_cellphone_holder" default="true" />
    <xacro:arg name="cellphone_holder_xyz" default="-0.021230953 0 0.05367" />
    <xacro:arg name="cellphone_holder_rpy" default="0 0 1.57079632679" />
@@ -37,5 +38,5 @@
      transmission_hw_interface="$(arg transmission_hw_interface)"
      sim="$(arg sim)"
-     basic_camera="$(arg basic_camera)"
+     basic_camera="$(arg left_basic_camera)"
      ip_address="$(arg left_ip_address)"
      verbose="$(arg verbose)"
@@ -59,5 +60,5 @@
      transmission_hw_interface="$(arg transmission_hw_interface)"
      sim="$(arg sim)"
-     basic_camera="$(arg basic_camera)"
+     basic_camera="$(arg right_basic_camera)"
      ip_address="$(arg right_ip_address)"
      verbose="$(arg verbose)"

Commit message: feat: add RealSense D405 touch tool and camera support to robot descriptions

File: denso_robot_descriptions/robots/vs050/urdf/denso_robot_macro.xacro (robot description, xacro)
@@ -64,5 +64,5 @@
       <xacro:include filename="$(find denso_robot_descriptions)/tools/basic_camera/urdf/basic_camera.xacro" />
     </xacro:if>
-    <xacro:if value="$(arg calib_tool)">
+    <xacro:if value="${calib_tool and not basic_camera}">
       <xacro:include filename="$(find denso_robot_descriptions)/tools/calibration_tool/urdf/calib.xacro" />
     </xacro:if>
@@ -100,12 +100,12 @@
       <xacro:basic_camera namespace="${namespace}" end_effector="J6" />
     </xacro:if>
-    <xacro:if value="$(arg calib_tool)">
+    <xacro:if value="${calib_tool and not basic_camera}">
       <xacro:calib
         namespace="${namespace}"
         end_effector="J6"
-        xyz="$(arg calib_xyz)"
-        rpy="$(arg calib_rpy)"
-        mesh_xyz="$(arg calib_mesh_xyz)"
-        mesh_rpy="$(arg calib_mesh_rpy)" />
+        xyz="${calib_xyz}"
+        rpy="${calib_rpy}"
+        mesh_xyz="${calib_mesh_xyz}"
+        mesh_rpy="${calib_mesh_rpy}" />
     </xacro:if>
     <xacro:if value="${cellphone_holder}">

File: denso_robot_descriptions/tools/basic_camera/urdf/basic_camera.xacro (robot description, xacro)
@@ -1,71 +1,120 @@
-<?xml version='1.0' encoding='UTF-8'?>
+<?xml version="1.0" encoding="UTF-8"?>
 <robot xmlns:xacro="http://www.ros.org/wiki/xacro">
-    <!-- here you define the parameters you want your xacro file to receive. -->
-    <xacro:macro name="basic_camera" params="namespace end_effector">
-    <!-- if your tool has meshes, define the path to it in geometry tag. -->
-    <!-- see the vs050 robot urdf implementation as an example. -->
-    <material name="${namespace}basic_camera_body_material">
-      <color rgba="0.05 0.16 0.30 1.0"/>
-    </material>
-    <material name="${namespace}basic_camera_view_axis_material">
-      <color rgba="0.0 0.75 1.0 0.55"/>
-    </material>
-    <link name="${namespace}basic_camera_link">
-		<inertial>
-			<mass value="1"/>
-			<inertia ixx="1" ixy="0" ixz="0" iyy="1" iyz="0" izz="1"/>
-		</inertial>
-		<collision>
-			<geometry>
-				<box size="0.035 0.03 0.025"/>
-			</geometry>
-		</collision>
-		<visual>
-			<geometry>
-				<box size="0.035 0.03 0.025"/>
-			</geometry>
-      <material name="${namespace}basic_camera_body_material"/>
-		</visual>
-	</link>
-  <link name="${namespace}basic_camera_view_axis">
-    <visual>
-      <origin rpy="0 1.57079632679 0" xyz="0.13 0 0"/>
-      <geometry>
-        <cylinder length="0.26" radius="0.003"/>
-      </geometry>
-      <material name="${namespace}basic_camera_view_axis_material"/>
-    </visual>
-  </link>
-  <joint name="${namespace}basic_camera_view_axis_joint" type="fixed">
-    <parent link="${namespace}basic_camera_link"/>
-    <child link="${namespace}basic_camera_view_axis"/>
-    <origin rpy="0 0 0" xyz="0 0 0"/>
-  </joint>
-	<joint name="${namespace}basic_camera_joint" type="fixed">
-        <!-- here you define where your tool will connect. In this case, it's at joint 6. -->
-		<parent link="${namespace}${end_effector}"/>
-		<child link="${namespace}basic_camera_link"/>
-		<origin rpy="0 ${radians(-90)} 0" xyz="0 0 0.01"/>
-	</joint>
+  <!-- Keep the basic_camera launch switch and RGB topic for existing clients.
+       Geometry and nominal D405 optics are documented in ../README.md. -->
+  <xacro:macro name="basic_camera" params="namespace end_effector">
+    <xacro:property name="d405_width" value="1280"/>
+    <xacro:property name="d405_height" value="720"/>
+    <!-- D400 datasheet (August 2025): D405 HD / 16:9 profile. -->
+    <xacro:property name="d405_hfov" value="${radians(84)}"/>
+    <xacro:property name="d405_vfov" value="${radians(58)}"/>
+    <link name="${namespace}toucher_link">
+      <!-- Estimated assembly mass / box inertia, not measured CAD dynamics. -->
+      <inertial>
+        <origin xyz="0 0.0188 0.025"/>
+        <mass value="0.16"/>
+        <inertia ixx="0.0001233" ixy="0" ixz="0"
+                 iyy="0.0000599" iyz="0" izz="0.0001165"/>
+      </inertial>
+      <visual>
+        <geometry>
+          <mesh filename="file:///$(find denso_robot_descriptions)/tools/basic_camera/meshes/toucher_with_realsense.stl"
+                scale="0.001 0.001 0.001"/>
+        </geometry>
+        <material name="${namespace}toucher_material">
+          <color rgba="0.65 0.65 0.68 1"/>
+        </material>
+      </visual>
+      <collision>
+        <geometry>
+          <mesh filename="file:///$(find denso_robot_descriptions)/tools/basic_camera/meshes/toucher_with_realsense.stl"
+                scale="0.001 0.001 0.001"/>
+        </geometry>
+      </collision>
+    </link>
+    <joint name="${namespace}toucher_joint" type="fixed">
+      <parent link="${namespace}${end_effector}"/>
+      <child link="${namespace}toucher_link"/>
+      <!-- CAD assembly is mounted 90 degrees counter-clockwise about J6. -->
+      <origin xyz="0 0 0" rpy="0 0 ${pi/2}"/>
+    </joint>
+    <!-- Keep the existing contact-frame name. Mounting Z=0; tip Z=50 mm. -->
+    <link name="${namespace}calib_link"/>
+    <joint name="${namespace}calib_joint" type="fixed">
+      <parent link="${namespace}toucher_link"/>
+      <child link="${namespace}calib_link"/>
+      <origin xyz="0 0 0.05" rpy="0 0 0"/>
+    </joint>
+    <!-- CAD front plate: (0, 38.876915, 27) mm. Nominal left imager:
+         -9 mm along tool X; zero depth is 3.8 mm behind the front plate.
+         Gazebo +X looks along tool +Z. The mounted imager's right/down
+         axes are tool -X/-Y: rotate the sensor roll, not the CAD assembly. -->
+    <link name="${namespace}basic_camera_link"/>
+    <joint name="${namespace}basic_camera_joint" type="fixed">
+      <parent link="${namespace}toucher_link"/>
+      <child link="${namespace}basic_camera_link"/>
+      <origin xyz="-0.009 0.038876915 0.0232" rpy="${-pi/2} ${-pi/2} 0"/>
+    </joint>
+    <link name="${namespace}camera_depth_optical_frame"/>
+    <joint name="${namespace}camera_depth_optical_joint" type="fixed">
+      <parent link="${namespace}basic_camera_link"/>
+      <child link="${namespace}camera_depth_optical_frame"/>
+      <origin xyz="0 0 0" rpy="${-pi/2} 0 ${-pi/2}"/>
+    </joint>
+    <!-- D405 color comes from the same left imager as depth. -->
+    <link name="${namespace}camera_color_optical_frame"/>
+    <joint name="${namespace}camera_color_optical_joint" type="fixed">
+      <parent link="${namespace}camera_depth_optical_frame"/>
+      <child link="${namespace}camera_color_optical_frame"/>
+      <origin xyz="0 0 0" rpy="0 0 0"/>
+    </joint>
+    <xacro:macro name="d405_sim_sensor" params="sensor_name sensor_type topic optical_frame near far info_topic">
+      <sensor name="${sensor_name}" type="${sensor_type}">
+        <always_on>true</always_on>
+        <update_rate>30</update_rate>
+        <visualize>true</visualize>
+        <topic>${topic}</topic>
+        <gz_frame_id>${optical_frame}</gz_frame_id>
+        <camera>
+          <horizontal_fov>${d405_hfov}</horizontal_fov>
+          <image>
+            <width>${d405_width}</width>
+            <height>${d405_height}</height>
+            <format>R8G8B8</format>
+          </image>
+          <clip><near>${near}</near><far>${far}</far></clip>
+          <!-- Set both focal lengths: aspect ratio alone would change VFOV. -->
+          <lens>
+            <type>gnomonical</type>
+            <intrinsics>
+              <fx>${d405_width / (2 * tan(d405_hfov / 2))}</fx>
+              <fy>${d405_height / (2 * tan(d405_vfov / 2))}</fy>
+              <cx>${d405_width / 2}</cx>
+              <cy>${d405_height / 2}</cy>
+              <s>0</s>
+            </intrinsics>
+            <projection>
+              <p_fx>${d405_width / (2 * tan(d405_hfov / 2))}</p_fx>
+              <p_fy>${d405_height / (2 * tan(d405_vfov / 2))}</p_fy>
+              <p_cx>${d405_width / 2}</p_cx>
+              <p_cy>${d405_height / 2}</p_cy>
+              <tx>0</tx><ty>0</ty>
+            </projection>
+          </lens>
+          <optical_frame_id>${optical_frame}</optical_frame_id>
+          <camera_info_topic>${info_topic}</camera_info_topic>
+        </camera>
+      </sensor>
+    </xacro:macro>
     <gazebo reference="${namespace}basic_camera_link">
-      <sensor name="${namespace}basic_camera" type="camera">
-        <camera>
-          <horizontal_fov>2.09439510239</horizontal_fov>
-          <image>
-            <width>640</width>
-            <height>480</height>
-          </image>
-          <clip>
-            <near>0.1</near>
-            <far>100</far>
-          </clip>
-        </camera>
-        <always_on>1</always_on>
-        <!-- Keep simulation and RViz responsive while preserving enough rate for alignment. -->
-        <update_rate>10</update_rate>
-        <visualize>true</visualize>
-        <topic>${namespace}basic_camera</topic>
-      </sensor>
+      <!-- RGB clipping is for rendering; 7–50 cm is the ideal DEPTH range. -->
+      <xacro:d405_sim_sensor sensor_name="${namespace}basic_camera" sensor_type="camera"
+        topic="${namespace}basic_camera" optical_frame="${namespace}camera_color_optical_frame"
+        near="0.005" far="100" info_topic="${namespace}basic_camera/camera_info"/>
+      <!-- A leaf image topic gives Gazebo DepthCameraSensor its own camera_info directory. -->
+      <xacro:d405_sim_sensor sensor_name="${namespace}d405_depth" sensor_type="depth_camera"
+        topic="${namespace}basic_camera/depth/image_raw" optical_frame="${namespace}camera_depth_optical_frame"
+        near="0.07" far="0.5" info_topic="${namespace}basic_camera/depth/camera_info"/>
     </gazebo>
-    </xacro:macro>
+  </xacro:macro>
 </robot>

File: denso_robot_moveit_config/robots/vs050/srdf/denso_robot_macro.srdf.xacro (robot description, xacro)
@@ -37,7 +37,5 @@
     </xacro:if>
     <xacro:if value="${basic_camera}">
-	  <disable_collisions link1="${namespace}J6" link2="${namespace}basic_camera_link" reason="Adjacent"/>
-	  <disable_collisions link1="${namespace}J5" link2="${namespace}basic_camera_link" reason="Never"/>
-	  <disable_collisions link1="${namespace}basic_camera_link" link2="${namespace}basic_camera_view_axis" reason="Adjacent"/>
+      <disable_collisions link1="${namespace}J6" link2="${namespace}toucher_link" reason="Adjacent"/>
     </xacro:if>
   </xacro:macro>

Commit message: feat: add virtual phone support with collision detection and parameters

File: denso_robot_descriptions/robots/vs050/urdf/denso_robot_macro.xacro (robot description, xacro)
@@ -29,4 +29,9 @@
     cellphone_holder_mesh_scale:='0.001 0.001 0.001'
     cellphone_holder_tag_size:=0.031
+    virtual_phone:=false
+    virtual_phone_width:=0.070
+    virtual_phone_height:=0.150
+    virtual_phone_thickness:=0.008
+    virtual_phone_screen_offset:=0.0
     ip_address
     send_format
@@ -118,5 +123,10 @@
         mesh_rpy="${cellphone_holder_mesh_rpy}"
         mesh_scale="${cellphone_holder_mesh_scale}"
-        tag_size="${cellphone_holder_tag_size}" />
+        tag_size="${cellphone_holder_tag_size}"
+        virtual_phone="${virtual_phone}"
+        virtual_phone_width="${virtual_phone_width}"
+        virtual_phone_height="${virtual_phone_height}"
+        virtual_phone_thickness="${virtual_phone_thickness}"
+        virtual_phone_screen_offset="${virtual_phone_screen_offset}" />
     </xacro:if>
   </xacro:macro>

File: denso_robot_descriptions/tools/basic_camera/urdf/basic_camera.xacro (robot description, xacro)
@@ -40,5 +40,11 @@
     </joint>
     <!-- Keep the existing contact-frame name. Mounting Z=0; tip Z=50 mm. -->
-    <link name="${namespace}calib_link"/>
+    <link name="${namespace}calib_link">
+      <!-- A small, named collision shape makes contact detection unambiguous.
+           The frame remains the existing physical touch TCP. -->
+      <collision name="${namespace}calib_contact">
+        <geometry><sphere radius="0.0015"/></geometry>
+      </collision>
+    </link>
     <joint name="${namespace}calib_joint" type="fixed">
       <parent link="${namespace}toucher_link"/>
@@ -46,4 +52,12 @@
       <origin xyz="0 0 0.05" rpy="0 0 0"/>
     </joint>
+    <gazebo reference="${namespace}calib_link">
+      <sensor name="${namespace}calib_contact_sensor" type="contact">
+        <always_on>true</always_on>
+        <update_rate>100</update_rate>
+        <topic>${namespace}calib_contact</topic>
+        <contact><collision>${namespace}calib_contact</collision></contact>
+      </sensor>
+    </gazebo>
     <!-- CAD front plate: (0, 38.876915, 27) mm. Nominal left imager:
          -9 mm along tool X; zero depth is 3.8 mm behind the front plate.

File: denso_robot_descriptions/tools/cellphone_holder/urdf/cellphone_holder.xacro (robot description, xacro)
@@ -54,5 +54,10 @@
     mesh_scale:='0.001 0.001 0.001'
     tag_size:=0.031
-    tag_thickness:=0.001">
+    tag_thickness:=0.001
+    virtual_phone:=false
+    virtual_phone_width:=0.070
+    virtual_phone_height:=0.150
+    virtual_phone_thickness:=0.008
+    virtual_phone_screen_offset:=0.0">
     <xacro:property name="top_tag_spacing" value="0.0952"/>
     <xacro:property name="bottom_tag_spacing" value="0.0998"/>
@@ -153,4 +158,44 @@
       tag_size="${tag_size}"
       tag_thickness="${tag_thickness}" />
+    <!-- The holder frame stays as the mechanical reference. The phone grows
+         along +Z, and the screen frame follows its outer contact surface. -->
+    <xacro:if value="${virtual_phone}">
+      <xacro:property name="virtual_phone_glass_thickness" value="0.001"/>
+      <xacro:property name="virtual_phone_body_thickness"
+                      value="${virtual_phone_thickness - virtual_phone_glass_thickness}"/>
+      <link name="${namespace}virtual_phone_link">
+        <visual name="phone_body_visual">
+          <origin xyz="0 0 ${virtual_phone_screen_offset + virtual_phone_body_thickness / 2.0}"/>
+          <geometry><box size="${virtual_phone_width} ${virtual_phone_height} ${virtual_phone_body_thickness}"/></geometry>
+          <material name="${namespace}virtual_phone_body_material"><color rgba="0.08 0.10 0.14 1"/></material>
+        </visual>
+        <collision name="${namespace}virtual_phone_body_collision">
+          <origin xyz="0 0 ${virtual_phone_screen_offset + virtual_phone_body_thickness / 2.0}"/>
+          <geometry><box size="${virtual_phone_width} ${virtual_phone_height} ${virtual_phone_body_thickness}"/></geometry>
+        </collision>
+      </link>
+      <joint name="${namespace}virtual_phone_joint" type="fixed">
+        <parent link="${namespace}cellphone_holder_phone_plane_frame"/>
+        <child link="${namespace}virtual_phone_link"/>
+        <origin xyz="0 0 0" rpy="0 0 0"/>
+      </joint>
+      <link name="${namespace}virtual_phone_screen_frame">
+        <visual name="screen_visual">
+          <!-- This link is the physical screen plane. The OBJ/MTL preserves
+               UV mapping in both RViz and Gazebo. -->
+          <origin xyz="0 0 0.00001" rpy="0 0 0"/>
+          <geometry><mesh filename="file://$(find denso_robot_descriptions)/tools/virtual_phone/meshes/phone_screen.obj" scale="${virtual_phone_height * 0.94} ${virtual_phone_height * 0.94} ${virtual_phone_height * 0.94}"/></geometry>
+        </visual>
+        <collision name="${namespace}virtual_phone_screen_collision">
+          <origin xyz="0 0 ${-virtual_phone_glass_thickness / 2.0}"/>
+          <geometry><box size="${virtual_phone_width * 0.94} ${virtual_phone_height * 0.94} ${virtual_phone_glass_thickness}"/></geometry>
+        </collision>
+      </link>
+      <joint name="${namespace}virtual_phone_screen_joint" type="fixed">
+        <parent link="${namespace}virtual_phone_link"/>
+        <child link="${namespace}virtual_phone_screen_frame"/>
+        <origin xyz="0 0 ${virtual_phone_screen_offset + virtual_phone_thickness}" rpy="0 0 0"/>
+      </joint>
+    </xacro:if>
   </xacro:macro>
 </robot>

File: denso_robot_descriptions/urdf/dual_denso_robot.urdf.xacro (robot description, xacro)
@@ -19,4 +19,10 @@
    <xacro:arg name="left_cellphone_holder" default="false" />
    <xacro:arg name="right_cellphone_holder" default="true" />
+   <xacro:arg name="left_virtual_phone" default="false" />
+   <xacro:arg name="right_virtual_phone" default="false" />
+   <xacro:arg name="virtual_phone_width" default="0.070" />
+   <xacro:arg name="virtual_phone_height" default="0.150" />
+   <xacro:arg name="virtual_phone_thickness" default="0.008" />
+   <xacro:arg name="virtual_phone_screen_offset" default="0.0" />
    <xacro:arg name="cellphone_holder_xyz" default="-0.021230953 0 0.05367" />
    <xacro:arg name="cellphone_holder_rpy" default="0 0 1.57079632679" />
@@ -50,5 +56,10 @@
      cellphone_holder_mesh_rpy="$(arg cellphone_holder_mesh_rpy)"
      cellphone_holder_mesh_scale="$(arg cellphone_holder_mesh_scale)"
-     cellphone_holder_tag_size="$(arg cellphone_holder_tag_size)" >
+     cellphone_holder_tag_size="$(arg cellphone_holder_tag_size)"
+     virtual_phone="$(arg left_virtual_phone)"
+     virtual_phone_width="$(arg virtual_phone_width)"
+     virtual_phone_height="$(arg virtual_phone_height)"
+     virtual_phone_thickness="$(arg virtual_phone_thickness)"
+     virtual_phone_screen_offset="$(arg virtual_phone_screen_offset)" >
      <origin xyz="$(arg left_xyz)" rpy="$(arg left_rpy)" />
    </xacro:denso_robot>
@@ -72,5 +83,10 @@
      cellphone_holder_mesh_rpy="$(arg cellphone_holder_mesh_rpy)"
      cellphone_holder_mesh_scale="$(arg cellphone_holder_mesh_scale)"
-     cellphone_holder_tag_size="$(arg cellphone_holder_tag_size)" >
+     cellphone_holder_tag_size="$(arg cellphone_holder_tag_size)"
+     virtual_phone="$(arg right_virtual_phone)"
+     virtual_phone_width="$(arg virtual_phone_width)"
+     virtual_phone_height="$(arg virtual_phone_height)"
+     virtual_phone_thickness="$(arg virtual_phone_thickness)"
+     virtual_phone_screen_offset="$(arg virtual_phone_screen_offset)" >
      <origin xyz="$(arg right_xyz)" rpy="$(arg right_rpy)" />
    </xacro:denso_robot>
