Commit message: Add cellphone collaboration vision workflow

File: denso_robot_descriptions/robots/vs050/urdf/denso_robot_macro.xacro (robot description, xacro)
@@ -28,5 +28,5 @@
     cellphone_holder_mesh_rpy:='0 0 1.57079632679'
     cellphone_holder_mesh_scale:='0.001 0.001 0.001'
-    cellphone_holder_tag_size:=0.031
+    cellphone_holder_tag_size:=0.026875
     virtual_phone:=false
     virtual_phone_width:=0.070

File: denso_robot_descriptions/tools/cellphone_holder/urdf/cellphone_holder.xacro (robot description, xacro)
@@ -8,17 +8,6 @@
     y
     z:=0
-    rpy:='0 0 0'
-    visual_radius:=0.004
-    color_rgba:='0.0 0.85 1.0 1.0'">
+    rpy:='0 0 0'">
     <link name="${namespace}${name}">
-      <visual>
-        <origin rpy="0 0 0" xyz="0 0 0"/>
-        <geometry>
-          <sphere radius="${visual_radius}"/>
-        </geometry>
-        <material name="${namespace}${name}_material">
-          <color rgba="${color_rgba}"/>
-        </material>
-      </visual>
     </link>
     <joint name="${namespace}${name}_joint" type="fixed">
@@ -28,5 +17,5 @@
     </joint>
   </xacro:macro>
-  <xacro:macro name="cellphone_holder_tag" params="namespace id x y tag_size tag_thickness">
+  <xacro:macro name="cellphone_holder_tag" params="namespace id x y tag_size tag_thickness rpy:='0 0 0'">
     <link name="${namespace}cellphone_holder_tag_${id}">
       <visual>
@@ -42,5 +31,5 @@
       <parent link="${namespace}cellphone_holder_tags_frame"/>
       <child link="${namespace}cellphone_holder_tag_${id}"/>
-      <origin rpy="0 0 0" xyz="${x} ${y} 0"/>
+      <origin rpy="${rpy}" xyz="${x} ${y} 0"/>
     </joint>
   </xacro:macro>
@@ -53,5 +42,5 @@
     mesh_rpy:='0 0 1.57079632679'
     mesh_scale:='0.001 0.001 0.001'
-    tag_size:=0.031
+    tag_size:=0.026875
     tag_thickness:=0.001
     virtual_phone:=false
@@ -103,7 +92,5 @@
       parent="${namespace}cellphone_holder_tags_frame"
       x="0"
-      y="0"
-      visual_radius="0.006"
-      color_rgba="1.0 0.85 0.0 1.0" />
+      y="0" />
     <xacro:cellphone_holder_reference_frame
       namespace="${namespace}"
@@ -136,5 +123,6 @@
       y="${side_tag_y_spacing / 2.0}"
       tag_size="${tag_size}"
-      tag_thickness="${tag_thickness}" />
+      tag_thickness="${tag_thickness}"
+      rpy="0 0 1.57079632679" />
     <xacro:cellphone_holder_tag
       namespace="${namespace}"
@@ -143,19 +131,22 @@
       y="${side_tag_y_spacing / 2.0}"
       tag_size="${tag_size}"
-      tag_thickness="${tag_thickness}" />
+      tag_thickness="${tag_thickness}"
+      rpy="0 0 -1.57079632679" />
     <xacro:cellphone_holder_tag
       namespace="${namespace}"
       id="3"
+      x="${bottom_tag_spacing / 2.0}"
+      y="${-side_tag_y_spacing / 2.0}"
+      tag_size="${tag_size}"
+      tag_thickness="${tag_thickness}"
+      rpy="0 0 1.57079632679" />
+    <xacro:cellphone_holder_tag
+      namespace="${namespace}"
+      id="4"
       x="${-bottom_tag_spacing / 2.0}"
       y="${-side_tag_y_spacing / 2.0}"
       tag_size="${tag_size}"
-      tag_thickness="${tag_thickness}" />
-    <xacro:cellphone_holder_tag
-      namespace="${namespace}"
-      id="4"
-      x="${bottom_tag_spacing / 2.0}"
-      y="${-side_tag_y_spacing / 2.0}"
-      tag_size="${tag_size}"
-      tag_thickness="${tag_thickness}" />
+      tag_thickness="${tag_thickness}"
+      rpy="0 0 1.57079632679" />
     <!-- The holder frame stays as the mechanical reference. The phone grows
          along +Z, and the screen frame follows its visible surface. -->
@@ -184,5 +175,5 @@
         </visual>
         <collision name="${namespace}virtual_phone_screen_collision">
-          <origin xyz="0 0 -0.0005"/>
+          <origin xyz="0 0 0.0006"/>
           <geometry><box size="${virtual_phone_width * 0.94} ${virtual_phone_height * 0.94} 0.001"/></geometry>
         </collision>

File: denso_robot_descriptions/urdf/dual_denso_robot.urdf.xacro (robot description, xacro)
@@ -30,5 +30,5 @@
    <xacro:arg name="cellphone_holder_mesh_rpy" default="0 0 1.57079632679" />
    <xacro:arg name="cellphone_holder_mesh_scale" default="0.001 0.001 0.001" />
-   <xacro:arg name="cellphone_holder_tag_size" default="0.031" />
+   <xacro:arg name="cellphone_holder_tag_size" default="0.026875" />
    <xacro:arg name="left_xyz" default="-0.4215124298776413 -0.0001916495678773618 -0.003297428813508002" />
    <xacro:arg name="left_rpy" default="0 0 0" />

Commit message: feat: add Hall touch D405 tool to single and dual DENSO models

File: denso_robot_descriptions/robots/vs050/urdf/denso_robot_macro.xacro (robot description, xacro)
@@ -17,4 +17,5 @@
     sim:=false
     basic_camera:=false
+    hall_touch_camera:=false
     calib_tool:=false
     calib_xyz:='0 0 0.05'
@@ -66,11 +67,14 @@
     <!-- The line with tag xacro:tool passes the parameters defined in your tool's xacro file -->
     <!-- (see basic_camera.xacro as an example implementation) -->
-    <xacro:if value="${basic_camera}">
+    <xacro:if value="${basic_camera and not hall_touch_camera}">
       <xacro:include filename="$(find denso_robot_descriptions)/tools/basic_camera/urdf/basic_camera.xacro" />
     </xacro:if>
-    <xacro:if value="${calib_tool and not basic_camera}">
+    <xacro:if value="${hall_touch_camera}">
+      <xacro:include filename="$(find denso_robot_descriptions)/tools/hall_touch_camera/urdf/hall_touch_camera.xacro" />
+    </xacro:if>
+    <xacro:if value="${calib_tool and not basic_camera and not hall_touch_camera}">
       <xacro:include filename="$(find denso_robot_descriptions)/tools/calibration_tool/urdf/calib.xacro" />
     </xacro:if>
-    <xacro:if value="${cellphone_holder}">
+    <xacro:if value="${cellphone_holder and not hall_touch_camera}">
       <xacro:include filename="$(find denso_robot_descriptions)/tools/cellphone_holder/urdf/cellphone_holder.xacro" />
     </xacro:if>
@@ -102,8 +106,11 @@
       <xacro:insert_block name="origin" />
     </xacro:denso_robot_arm_kinematics>
-    <xacro:if value="${basic_camera}">
+    <xacro:if value="${basic_camera and not hall_touch_camera}">
       <xacro:basic_camera namespace="${namespace}" end_effector="J6" />
     </xacro:if>
-    <xacro:if value="${calib_tool and not basic_camera}">
+    <xacro:if value="${hall_touch_camera}">
+      <xacro:hall_touch_camera namespace="${namespace}" end_effector="J6" />
+    </xacro:if>
+    <xacro:if value="${calib_tool and not basic_camera and not hall_touch_camera}">
       <xacro:calib
         namespace="${namespace}"
@@ -114,5 +121,5 @@
         mesh_rpy="${calib_mesh_rpy}" />
     </xacro:if>
-    <xacro:if value="${cellphone_holder}">
+    <xacro:if value="${cellphone_holder and not hall_touch_camera}">
       <xacro:cellphone_holder
         namespace="${namespace}"

File: denso_robot_descriptions/robots/vs060/urdf/denso_robot_macro.xacro (robot description, xacro)
@@ -17,4 +17,5 @@
     sim:=false
     basic_camera:=false
+    hall_touch_camera:=false
     calib_tool:=false
     calib_xyz:='0 0 0.05'
@@ -29,4 +30,9 @@
     cellphone_holder_mesh_scale:='0.001 0.001 0.001'
     cellphone_holder_tag_size:=0.031
+    virtual_phone:=false
+    virtual_phone_width:=0.070
+    virtual_phone_height:=0.150
+    virtual_phone_thickness:=0.008
+    virtual_phone_screen_offset:=0.0
     ip_address
     send_format
@@ -61,11 +67,14 @@
     <!-- The line with tag xacro:tool passes the parameters defined in your tool's xacro file -->
     <!-- (see basic_camera.xacro as an example implementation) -->
-    <xacro:if value="${basic_camera}">
+    <xacro:if value="${basic_camera and not hall_touch_camera}">
       <xacro:include filename="$(find denso_robot_descriptions)/tools/basic_camera/urdf/basic_camera.xacro" />
     </xacro:if>
-    <xacro:if value="${calib_tool}">
+    <xacro:if value="${hall_touch_camera}">
+      <xacro:include filename="$(find denso_robot_descriptions)/tools/hall_touch_camera/urdf/hall_touch_camera.xacro" />
+    </xacro:if>
+    <xacro:if value="${calib_tool and not basic_camera and not hall_touch_camera}">
       <xacro:include filename="$(find denso_robot_descriptions)/tools/calibration_tool/urdf/calib.xacro" />
     </xacro:if>
-    <xacro:if value="${cellphone_holder}">
+    <xacro:if value="${cellphone_holder and not hall_touch_camera}">
       <xacro:include filename="$(find denso_robot_descriptions)/tools/cellphone_holder/urdf/cellphone_holder.xacro" />
     </xacro:if>
@@ -97,8 +106,11 @@
       <xacro:insert_block name="origin" />
     </xacro:denso_robot_arm_kinematics>
-    <xacro:if value="${basic_camera}">
+    <xacro:if value="${basic_camera and not hall_touch_camera}">
       <xacro:basic_camera namespace="${namespace}" end_effector="J6" />
     </xacro:if>
-    <xacro:if value="${calib_tool}">
+    <xacro:if value="${hall_touch_camera}">
+      <xacro:hall_touch_camera namespace="${namespace}" end_effector="J6" />
+    </xacro:if>
+    <xacro:if value="${calib_tool and not basic_camera and not hall_touch_camera}">
       <xacro:calib
         namespace="${namespace}"
@@ -109,5 +121,5 @@
         mesh_rpy="${calib_mesh_rpy}" />
     </xacro:if>
-    <xacro:if value="${cellphone_holder}">
+    <xacro:if value="${cellphone_holder and not hall_touch_camera}">
       <xacro:cellphone_holder
         namespace="${namespace}"

File: denso_robot_descriptions/urdf/denso_robot.urdf.xacro (robot description, xacro)
@@ -12,4 +12,5 @@
    <xacro:arg name="sim" default="false" />
    <xacro:arg name="basic_camera" default="false" />
+   <xacro:arg name="hall_touch_camera" default="false" />
   <xacro:arg name="calib_tool" default="false" />
   <xacro:arg name="calib_xyz" default="0 0 0.05" />
@@ -39,4 +40,5 @@
      sim="$(arg sim)"
      basic_camera="$(arg basic_camera)"
+     hall_touch_camera="$(arg hall_touch_camera)"
     calib_tool="$(arg calib_tool)"
     calib_xyz="$(arg calib_xyz)"

File: denso_robot_descriptions/urdf/dual_denso_robot.urdf.xacro (robot description, xacro)
@@ -12,4 +12,6 @@
    <xacro:arg name="left_basic_camera" default="true" />
    <xacro:arg name="right_basic_camera" default="false" />
+   <xacro:arg name="left_hall_touch_camera" default="false" />
+   <xacro:arg name="right_hall_touch_camera" default="false" />
    <xacro:arg name="left_ip_address" default="192.168.0.1" />
    <xacro:arg name="right_ip_address" default="192.168.0.2" />
@@ -45,4 +47,5 @@
      sim="$(arg sim)"
      basic_camera="$(arg left_basic_camera)"
+     hall_touch_camera="$(arg left_hall_touch_camera)"
      ip_address="$(arg left_ip_address)"
      verbose="$(arg verbose)"
@@ -72,4 +75,5 @@
      sim="$(arg sim)"
      basic_camera="$(arg right_basic_camera)"
+     hall_touch_camera="$(arg right_hall_touch_camera)"
      ip_address="$(arg right_ip_address)"
      verbose="$(arg verbose)"

File: denso_robot_moveit_config/robots/vs050/srdf/denso_robot_macro.srdf.xacro (robot description, xacro)
@@ -5,5 +5,5 @@
     A URDF file must exist for this robot as well, where the joints and the links that are referenced are defined
 -->
-	<xacro:macro name="denso_robot_srdf" params="namespace calib_tool:=false basic_camera:=false">
+	<xacro:macro name="denso_robot_srdf" params="namespace calib_tool:=false basic_camera:=false hall_touch_camera:=false">
     <!--GROUPS - Representation of a set of joints and links. This can be useful for specifying DOF to plan for, defining arms, end effectors, etc-->
     <!--LINKS - When a link is specified, the parent joint of that link (if it exists) is automatically included-->
@@ -32,10 +32,13 @@
 	<disable_collisions link1="${namespace}J3" link2="${namespace}J5" reason="Never"/>
 	<disable_collisions link1="${namespace}J4" link2="${namespace}J5" reason="Adjacent"/>
-    <xacro:if value="${calib_tool}">
+    <xacro:if value="${calib_tool and not basic_camera and not hall_touch_camera}">
 	  <disable_collisions link1="${namespace}J6" link2="${namespace}calib_link" reason="Adjacent"/>
 	  <disable_collisions link1="${namespace}J5" link2="${namespace}calib_link" reason="Never"/>
     </xacro:if>
-    <xacro:if value="${basic_camera}">
+    <xacro:if value="${basic_camera and not hall_touch_camera}">
       <disable_collisions link1="${namespace}J6" link2="${namespace}toucher_link" reason="Adjacent"/>
+    </xacro:if>
+    <xacro:if value="${hall_touch_camera}">
+      <disable_collisions link1="${namespace}J6" link2="${namespace}hall_camera_support_link" reason="Adjacent"/>
     </xacro:if>
   </xacro:macro>

File: denso_robot_moveit_config/robots/vs060/srdf/denso_robot_macro.srdf.xacro (robot description, xacro)
@@ -5,5 +5,5 @@
     A URDF file must exist for this robot as well, where the joints and the links that are referenced are defined
 -->
-  <xacro:macro name="denso_robot_srdf" params="namespace">
+  <xacro:macro name="denso_robot_srdf" params="namespace calib_tool:=false basic_camera:=false hall_touch_camera:=false">
     <!--GROUPS - Representation of a set of joints and links. This can be useful for specifying DOF to plan for, defining arms, end effectors, etc-->
     <!--LINKS - When a link is specified, the parent joint of that link (if it exists) is automatically included-->
@@ -32,4 +32,7 @@
 	<disable_collisions link1="${namespace}J3" link2="${namespace}J5" reason="Never"/>
 	<disable_collisions link1="${namespace}J4" link2="${namespace}J5" reason="Adjacent"/>
+    <xacro:if value="${hall_touch_camera}">
+      <disable_collisions link1="${namespace}J6" link2="${namespace}hall_camera_support_link" reason="Adjacent"/>
+    </xacro:if>
   </xacro:macro>
 </robot>

File: denso_robot_moveit_config/srdf/denso_robot.srdf.xacro (robot description, xacro)
@@ -6,5 +6,8 @@
   <xacro:arg name="namespace" default="" />
   <xacro:arg name="calib_tool" default="false" />
+  <xacro:arg name="basic_camera" default="false" />
+  <xacro:arg name="hall_touch_camera" default="false" />
   <xacro:include filename="$(find denso_robot_moveit_config)/robots/$(arg model)/srdf/denso_robot_macro.srdf.xacro"/>
-  <xacro:denso_robot_srdf namespace="$(arg namespace)" calib_tool="$(arg calib_tool)"/>
+  <xacro:denso_robot_srdf namespace="$(arg namespace)" calib_tool="$(arg calib_tool)"
+    basic_camera="$(arg basic_camera)" hall_touch_camera="$(arg hall_touch_camera)"/>
 </robot>

File: denso_robot_moveit_config/srdf/dual_denso_robot.srdf.xacro (robot description, xacro)
@@ -6,9 +6,13 @@
   <xacro:arg name="right_basic_camera" default="false"/>
   <xacro:arg name="right_virtual_phone" default="false"/>
+  <xacro:arg name="left_hall_touch_camera" default="false"/>
+  <xacro:arg name="right_hall_touch_camera" default="false"/>
   <xacro:include filename="$(find denso_robot_moveit_config)/robots/$(arg model)/srdf/denso_robot_macro.srdf.xacro"/>
   <!-- left arm -->
-  <xacro:denso_robot_srdf namespace="left_" basic_camera="$(arg left_basic_camera)"/>
+  <xacro:denso_robot_srdf namespace="left_" basic_camera="$(arg left_basic_camera)"
+    hall_touch_camera="$(arg left_hall_touch_camera)"/>
   <!-- right arm -->
-  <xacro:denso_robot_srdf namespace="right_" basic_camera="$(arg right_basic_camera)"/>
+  <xacro:denso_robot_srdf namespace="right_" basic_camera="$(arg right_basic_camera)"
+    hall_touch_camera="$(arg right_hall_touch_camera)"/>
   <group name="dual_arm">
     <group name="left_arm"/>

Commit message: Configure Hall tool calibration in robot bringup

File: denso_robot_descriptions/robots/vs050/urdf/denso_robot_macro.xacro (robot description, xacro)
@@ -18,4 +18,6 @@
     basic_camera:=false
     hall_touch_camera:=false
+    hall_touch_calib_offset_x_mm:=-2
+    hall_touch_calib_offset_y_mm:=-1
     calib_tool:=false
     calib_xyz:='0 0 0.05'
@@ -110,5 +112,9 @@
     </xacro:if>
     <xacro:if value="${hall_touch_camera}">
-      <xacro:hall_touch_camera namespace="${namespace}" end_effector="J6" />
+      <xacro:hall_touch_camera
+        namespace="${namespace}"
+        end_effector="J6"
+        calib_offset_x_mm="${hall_touch_calib_offset_x_mm}"
+        calib_offset_y_mm="${hall_touch_calib_offset_y_mm}" />
     </xacro:if>
     <xacro:if value="${calib_tool and not basic_camera and not hall_touch_camera}">

File: denso_robot_descriptions/robots/vs060/urdf/denso_robot_macro.xacro (robot description, xacro)
@@ -18,4 +18,6 @@
     basic_camera:=false
     hall_touch_camera:=false
+    hall_touch_calib_offset_x_mm:=-2
+    hall_touch_calib_offset_y_mm:=-1
     calib_tool:=false
     calib_xyz:='0 0 0.05'
@@ -110,5 +112,9 @@
     </xacro:if>
     <xacro:if value="${hall_touch_camera}">
-      <xacro:hall_touch_camera namespace="${namespace}" end_effector="J6" />
+      <xacro:hall_touch_camera
+        namespace="${namespace}"
+        end_effector="J6"
+        calib_offset_x_mm="${hall_touch_calib_offset_x_mm}"
+        calib_offset_y_mm="${hall_touch_calib_offset_y_mm}" />
     </xacro:if>
     <xacro:if value="${calib_tool and not basic_camera and not hall_touch_camera}">

File: denso_robot_descriptions/tools/hall_touch_camera/urdf/hall_touch_camera.xacro (robot description, xacro)
@@ -3,5 +3,9 @@
   <!-- Fusion coordinates are millimetres with the mounting face at J6.
        The three links are the camera support, touch TCP, and left optical centre. -->
-  <xacro:macro name="hall_touch_camera" params="namespace end_effector">
+  <xacro:macro name="hall_touch_camera" params="
+    namespace
+    end_effector
+    calib_offset_x_mm:=-2
+    calib_offset_y_mm:=-1">
     <xacro:property name="d405_width" value="1920"/>
     <xacro:property name="d405_height" value="1080"/>
@@ -49,5 +53,10 @@
       <parent link="${namespace}hall_camera_support_link"/>
       <child link="${namespace}calib_link"/>
-      <origin xyz="0 0 0.105987" rpy="0 0 ${pi}"/>
+      <!-- Offsets are expressed in calib_link's local X/Y axes and exposed
+           in millimetres. The joint origin translation is expressed in the
+           parent frame, so local Y changes sign after the pi rotation in X. -->
+      <origin
+        xyz="${calib_offset_x_mm * 0.001} ${-calib_offset_y_mm * 0.001} 0.105987"
+        rpy="0 0 ${pi}"/>
     </joint>
     <!-- Nominal D405 left imager: half the 18.047 mm stereo baseline in

File: denso_robot_descriptions/urdf/denso_robot.urdf.xacro (robot description, xacro)
@@ -13,4 +13,6 @@
    <xacro:arg name="basic_camera" default="false" />
    <xacro:arg name="hall_touch_camera" default="false" />
+   <xacro:arg name="hall_touch_calib_offset_x_mm" default="-2" />
+   <xacro:arg name="hall_touch_calib_offset_y_mm" default="-1" />
   <xacro:arg name="calib_tool" default="false" />
   <xacro:arg name="calib_xyz" default="0 0 0.05" />
@@ -41,4 +43,6 @@
      basic_camera="$(arg basic_camera)"
      hall_touch_camera="$(arg hall_touch_camera)"
+     hall_touch_calib_offset_x_mm="$(arg hall_touch_calib_offset_x_mm)"
+     hall_touch_calib_offset_y_mm="$(arg hall_touch_calib_offset_y_mm)"
     calib_tool="$(arg calib_tool)"
     calib_xyz="$(arg calib_xyz)"

File: denso_robot_descriptions/urdf/dual_denso_robot.urdf.xacro (robot description, xacro)
@@ -14,4 +14,8 @@
    <xacro:arg name="left_hall_touch_camera" default="false" />
    <xacro:arg name="right_hall_touch_camera" default="false" />
+   <xacro:arg name="left_hall_touch_calib_offset_x_mm" default="-2" />
+   <xacro:arg name="left_hall_touch_calib_offset_y_mm" default="-1" />
+   <xacro:arg name="right_hall_touch_calib_offset_x_mm" default="0" />
+   <xacro:arg name="right_hall_touch_calib_offset_y_mm" default="0" />
    <xacro:arg name="left_ip_address" default="192.168.160.228" />
    <xacro:arg name="right_ip_address" default="192.168.160.227" />
@@ -48,4 +52,6 @@
      basic_camera="$(arg left_basic_camera)"
      hall_touch_camera="$(arg left_hall_touch_camera)"
+     hall_touch_calib_offset_x_mm="$(arg left_hall_touch_calib_offset_x_mm)"
+     hall_touch_calib_offset_y_mm="$(arg left_hall_touch_calib_offset_y_mm)"
      ip_address="$(arg left_ip_address)"
      verbose="$(arg verbose)"
@@ -76,4 +82,6 @@
      basic_camera="$(arg right_basic_camera)"
      hall_touch_camera="$(arg right_hall_touch_camera)"
+     hall_touch_calib_offset_x_mm="$(arg right_hall_touch_calib_offset_x_mm)"
+     hall_touch_calib_offset_y_mm="$(arg right_hall_touch_calib_offset_y_mm)"
      ip_address="$(arg right_ip_address)"
      verbose="$(arg verbose)"
