Commit message: Add CAPTCHA collaboration targets and separate test guides

File: denso_robot_descriptions/robots/vs050/urdf/denso_robot_macro.xacro (robot description, xacro)
@@ -33,4 +33,5 @@
     cellphone_holder_tag_size:=0.026875
     virtual_phone:=false
+    virtual_phone_target:=rgb
     virtual_phone_width:=0.070
     virtual_phone_height:=0.150
@@ -138,4 +139,5 @@
         tag_size="${cellphone_holder_tag_size}"
         virtual_phone="${virtual_phone}"
+        virtual_phone_target="${virtual_phone_target}"
         virtual_phone_width="${virtual_phone_width}"
         virtual_phone_height="${virtual_phone_height}"

File: denso_robot_descriptions/robots/vs060/urdf/denso_robot_macro.xacro (robot description, xacro)
@@ -33,4 +33,5 @@
     cellphone_holder_tag_size:=0.031
     virtual_phone:=false
+    virtual_phone_target:=rgb
     virtual_phone_width:=0.070
     virtual_phone_height:=0.150

File: denso_robot_descriptions/tools/cellphone_holder/urdf/cellphone_holder.xacro (robot description, xacro)
@@ -45,4 +45,5 @@
     tag_thickness:=0.001
     virtual_phone:=false
+    virtual_phone_target:=rgb
     virtual_phone_width:=0.070
     virtual_phone_height:=0.150
@@ -180,5 +181,5 @@
           <!-- The OBJ/MTL preserves UV mapping in RViz and Gazebo. -->
           <origin xyz="0 0 0.00001" rpy="0 0 0"/>
-          <geometry><mesh filename="file://$(find denso_robot_descriptions)/tools/virtual_phone/meshes/phone_screen.obj" scale="${virtual_phone_height * 0.94} ${virtual_phone_height * 0.94} ${virtual_phone_height * 0.94}"/></geometry>
+          <geometry><mesh filename="file://$(find denso_robot_descriptions)/tools/virtual_phone/meshes/${dict(rgb='phone_screen', captcha='phone_captcha')[virtual_phone_target]}.obj" scale="${virtual_phone_height * 0.94} ${virtual_phone_height * 0.94} ${virtual_phone_height * 0.94}"/></geometry>
         </visual>
         <collision name="${namespace}virtual_phone_screen_collision">

File: denso_robot_descriptions/urdf/dual_denso_robot.urdf.xacro (robot description, xacro)
@@ -27,4 +27,5 @@
    <xacro:arg name="left_virtual_phone" default="false" />
    <xacro:arg name="right_virtual_phone" default="false" />
+   <xacro:arg name="target" default="rgb" />
    <xacro:arg name="virtual_phone_width" default="0.070" />
    <xacro:arg name="virtual_phone_height" default="0.150" />
@@ -67,4 +68,5 @@
      cellphone_holder_tag_size="$(arg cellphone_holder_tag_size)"
      virtual_phone="$(arg left_virtual_phone)"
+     virtual_phone_target="$(arg target)"
      virtual_phone_width="$(arg virtual_phone_width)"
      virtual_phone_height="$(arg virtual_phone_height)"
@@ -97,4 +99,5 @@
      cellphone_holder_tag_size="$(arg cellphone_holder_tag_size)"
      virtual_phone="$(arg right_virtual_phone)"
+     virtual_phone_target="$(arg target)"
      virtual_phone_width="$(arg virtual_phone_width)"
      virtual_phone_height="$(arg virtual_phone_height)"
