Commit message: fix(calib): update mesh scale in collision and visual sections to 1 1 1 for proper rendering

File: denso_robot_descriptions/tools/calibration_tool/urdf/calib.xacro (robot description, xacro)
@@ -11,5 +11,5 @@
 			<origin rpy="${mesh_rpy}" xyz="${mesh_xyz}"/>
 			<geometry>
-				<mesh filename="file:///$(find denso_robot_descriptions)/tools/calibration_tool/meshes/calibration_tool.dae" scale="0.001 0.001 0.001"/>
+				<mesh filename="file:///$(find denso_robot_descriptions)/tools/calibration_tool/meshes/calibration_tool.dae" scale="1 1 1"/>
 			</geometry>
 		</collision>
@@ -17,5 +17,5 @@
 			<origin rpy="${mesh_rpy}" xyz="${mesh_xyz}"/>
 			<geometry>
-				<mesh filename="file:///$(find denso_robot_descriptions)/tools/calibration_tool/meshes/calibration_tool.dae" scale="0.001 0.001 0.001"/>
+				<mesh filename="file:///$(find denso_robot_descriptions)/tools/calibration_tool/meshes/calibration_tool.dae" scale="1 1 1"/>
 			</geometry>
 		</visual>

Commit message: fix(calib): add missing material section in visual element for calibration tool

File: denso_robot_descriptions/tools/calibration_tool/urdf/calib.xacro (robot description, xacro)
@@ -15,4 +15,7 @@
 		</collision>
 		<visual>
+			<material name="calib_material">
+				<color rgba="0.8 0.1 0.1 1"/>
+			</material>
 			<origin rpy="${mesh_rpy}" xyz="${mesh_xyz}"/>
 			<geometry>
