Commit message: fix reference point to match opencv detection of arucos

File: denso_robot_descriptions/tools/cellphone_holder/urdf/cellphone_holder.xacro (robot description, xacro)
@@ -1,4 +1,31 @@
 <?xml version='1.0' encoding='UTF-8'?>
 <robot xmlns:xacro="http://www.ros.org/wiki/xacro">
+  <xacro:macro name="cellphone_holder_reference_frame" params="
+    namespace
+    name
+    parent
+    x
+    y
+    z:=0
+    rpy:='0 0 0'
+    visual_radius:=0.004
+    color_rgba:='0.0 0.85 1.0 1.0'">
+    <link name="${namespace}${name}">
+      <visual>
+        <origin rpy="0 0 0" xyz="0 0 0"/>
+        <geometry>
+          <sphere radius="${visual_radius}"/>
+        </geometry>
+        <material name="${namespace}${name}_material">
+          <color rgba="${color_rgba}"/>
+        </material>
+      </visual>
+    </link>
+    <joint name="${namespace}${name}_joint" type="fixed">
+      <parent link="${parent}"/>
+      <child link="${namespace}${name}"/>
+      <origin rpy="${rpy}" xyz="${x} ${y} ${z}"/>
+    </joint>
+  </xacro:macro>
   <xacro:macro name="cellphone_holder_tag" params="namespace id x y tag_size tag_thickness">
     <link name="${namespace}cellphone_holder_tag_${id}">
@@ -32,4 +59,8 @@
     <xacro:property name="side_tag_spacing" value="0.2075"/>
     <xacro:property name="side_tag_y_spacing" value="0.2074872534"/>
+    <xacro:property name="detected_tag_size" value="${tag_size * 0.8}"/>
+    <xacro:property name="top_tag_detected_outer_x" value="${top_tag_spacing / 2.0 + detected_tag_size / 2.0}"/>
+    <xacro:property name="bottom_tag_detected_outer_x" value="${bottom_tag_spacing / 2.0 + detected_tag_size / 2.0}"/>
+    <xacro:property name="tag_detected_outer_y" value="${side_tag_y_spacing / 2.0 + detected_tag_size / 2.0}"/>
     <link name="${namespace}cellphone_holder_mount_frame">
       <visual>
@@ -50,10 +81,48 @@
       <origin rpy="0 0 0" xyz="0 0 0"/>
     </joint>
-    <link name="${namespace}cellphone_holder_tags_frame"/>
+    <link name="${namespace}cellphone_holder_phone_plane_frame"/>
     <joint name="${namespace}cellphone_holder_joint" type="fixed">
       <parent link="${namespace}cellphone_holder_mount_frame"/>
-      <child link="${namespace}cellphone_holder_tags_frame"/>
+      <child link="${namespace}cellphone_holder_phone_plane_frame"/>
       <origin rpy="${rpy}" xyz="${xyz}"/>
     </joint>
+    <link name="${namespace}cellphone_holder_tags_frame"/>
+    <joint name="${namespace}cellphone_holder_tags_frame_joint" type="fixed">
+      <parent link="${namespace}cellphone_holder_phone_plane_frame"/>
+      <child link="${namespace}cellphone_holder_tags_frame"/>
+      <origin rpy="0 0 0" xyz="0 0 0"/>
+    </joint>
+    <xacro:cellphone_holder_reference_frame
+      namespace="${namespace}"
+      name="cellphone_holder_tag_rectangle_center_frame"
+      parent="${namespace}cellphone_holder_tags_frame"
+      x="0"
+      y="0"
+      visual_radius="0.006"
+      color_rgba="1.0 0.85 0.0 1.0" />
+    <xacro:cellphone_holder_reference_frame
+      namespace="${namespace}"
+      name="cellphone_holder_ref_upper_left"
+      parent="${namespace}cellphone_holder_tags_frame"
+      x="${-top_tag_detected_outer_x}"
+      y="${tag_detected_outer_y}" />
+    <xacro:cellphone_holder_reference_frame
+      namespace="${namespace}"
+      name="cellphone_holder_ref_upper_right"
+      parent="${namespace}cellphone_holder_tags_frame"
+      x="${top_tag_detected_outer_x}"
+      y="${tag_detected_outer_y}" />
+    <xacro:cellphone_holder_reference_frame
+      namespace="${namespace}"
+      name="cellphone_holder_ref_lower_left"
+      parent="${namespace}cellphone_holder_tags_frame"
+      x="${-bottom_tag_detected_outer_x}"
+      y="${-tag_detected_outer_y}" />
+    <xacro:cellphone_holder_reference_frame
+      namespace="${namespace}"
+      name="cellphone_holder_ref_lower_right"
+      parent="${namespace}cellphone_holder_tags_frame"
+      x="${bottom_tag_detected_outer_x}"
+      y="${-tag_detected_outer_y}" />
     <xacro:cellphone_holder_tag
       namespace="${namespace}"

Commit message: fix: restore virtual phone collision geometry

File: denso_robot_descriptions/tools/cellphone_holder/urdf/cellphone_holder.xacro (robot description, xacro)
@@ -167,4 +167,8 @@
           <material name="${namespace}virtual_phone_body_material"><color rgba="0.08 0.10 0.14 1"/></material>
         </visual>
+        <collision name="${namespace}virtual_phone_body_collision">
+          <origin xyz="0 0 ${virtual_phone_screen_offset + virtual_phone_thickness / 2.0}"/>
+          <geometry><box size="${virtual_phone_width} ${virtual_phone_height} ${virtual_phone_thickness}"/></geometry>
+        </collision>
       </link>
       <joint name="${namespace}virtual_phone_joint" type="fixed">
@@ -179,4 +183,8 @@
           <geometry><mesh filename="file://$(find denso_robot_descriptions)/tools/virtual_phone/meshes/phone_screen.obj" scale="${virtual_phone_height * 0.94} ${virtual_phone_height * 0.94} ${virtual_phone_height * 0.94}"/></geometry>
         </visual>
+        <collision name="${namespace}virtual_phone_screen_collision">
+          <origin xyz="0 0 -0.0005"/>
+          <geometry><box size="${virtual_phone_width * 0.94} ${virtual_phone_height * 0.94} 0.001"/></geometry>
+        </collision>
       </link>
       <joint name="${namespace}virtual_phone_screen_joint" type="fixed">

Commit message: fix: add cellphone holder collision geometry

File: denso_robot_descriptions/tools/cellphone_holder/urdf/cellphone_holder.xacro (robot description, xacro)
@@ -69,4 +69,12 @@
         </material>
       </visual>
+      <collision>
+        <origin rpy="${mesh_rpy}" xyz="${mesh_xyz}"/>
+        <geometry>
+          <mesh
+            filename="file://$(find denso_robot_descriptions)/tools/cellphone_holder/meshes/cellphone_holder.stl"
+            scale="${mesh_scale}"/>
+        </geometry>
+      </collision>
     </link>
     <joint name="${namespace}cellphone_holder_mount_joint" type="fixed">
