Commit message: Fix MoveIt camera self-collision semantics

File: denso_robot_moveit_config/robots/vs050/srdf/denso_robot_macro.srdf.xacro (robot description, xacro)
@@ -5,5 +5,5 @@
     A URDF file must exist for this robot as well, where the joints and the links that are referenced are defined
 -->
-	<xacro:macro name="denso_robot_srdf" params="namespace calib_tool:=false">
+	<xacro:macro name="denso_robot_srdf" params="namespace calib_tool:=false basic_camera:=false">
     <!--GROUPS - Representation of a set of joints and links. This can be useful for specifying DOF to plan for, defining arms, end effectors, etc-->
     <!--LINKS - When a link is specified, the parent joint of that link (if it exists) is automatically included-->
@@ -36,4 +36,9 @@
 	  <disable_collisions link1="${namespace}J5" link2="${namespace}calib_link" reason="Never"/>
     </xacro:if>
+    <xacro:if value="${basic_camera}">
+	  <disable_collisions link1="${namespace}J6" link2="${namespace}basic_camera_link" reason="Adjacent"/>
+	  <disable_collisions link1="${namespace}J5" link2="${namespace}basic_camera_link" reason="Never"/>
+	  <disable_collisions link1="${namespace}basic_camera_link" link2="${namespace}basic_camera_view_axis" reason="Adjacent"/>
+    </xacro:if>
   </xacro:macro>
 </robot>

File: denso_robot_moveit_config/srdf/dual_denso_robot.srdf.xacro (robot description, xacro)
@@ -3,9 +3,11 @@
   <!-- robot name parameter -->
   <xacro:arg name="model" default="denso_robot"/>
+  <xacro:arg name="left_basic_camera" default="true"/>
+  <xacro:arg name="right_basic_camera" default="false"/>
   <xacro:include filename="$(find denso_robot_moveit_config)/robots/$(arg model)/srdf/denso_robot_macro.srdf.xacro"/>
   <!-- left arm -->
-  <xacro:denso_robot_srdf namespace="left_"/>
+  <xacro:denso_robot_srdf namespace="left_" basic_camera="$(arg left_basic_camera)"/>
   <!-- right arm -->
-  <xacro:denso_robot_srdf namespace="right_"/>
+  <xacro:denso_robot_srdf namespace="right_" basic_camera="$(arg right_basic_camera)"/>
   <group name="dual_arm">
     <group name="left_arm"/>
