Commit message: refactor: defer virtual phone contact simulation

File: denso_robot_descriptions/tools/basic_camera/urdf/basic_camera.xacro (robot description, xacro)
@@ -40,11 +40,5 @@
     </joint>
     <!-- Keep the existing contact-frame name. Mounting Z=0; tip Z=50 mm. -->
-    <link name="${namespace}calib_link">
-      <!-- A small, named collision shape makes contact detection unambiguous.
-           The frame remains the existing physical touch TCP. -->
-      <collision name="${namespace}calib_contact">
-        <geometry><sphere radius="0.0015"/></geometry>
-      </collision>
-    </link>
+    <link name="${namespace}calib_link"/>
     <joint name="${namespace}calib_joint" type="fixed">
       <parent link="${namespace}toucher_link"/>
@@ -52,12 +46,4 @@
       <origin xyz="0 0 0.05" rpy="0 0 0"/>
     </joint>
-    <gazebo reference="${namespace}calib_link">
-      <sensor name="${namespace}calib_contact_sensor" type="contact">
-        <always_on>true</always_on>
-        <update_rate>100</update_rate>
-        <topic>${namespace}calib_contact</topic>
-        <contact><collision>${namespace}calib_contact</collision></contact>
-      </sensor>
-    </gazebo>
     <!-- CAD front plate: (0, 38.876915, 27) mm. Nominal left imager:
          -9 mm along tool X; zero depth is 3.8 mm behind the front plate.

File: denso_robot_descriptions/tools/cellphone_holder/urdf/cellphone_holder.xacro (robot description, xacro)
@@ -159,19 +159,12 @@
       tag_thickness="${tag_thickness}" />
     <!-- The holder frame stays as the mechanical reference. The phone grows
-         along +Z, and the screen frame follows its outer contact surface. -->
+         along +Z, and the screen frame follows its visible surface. -->
     <xacro:if value="${virtual_phone}">
-      <xacro:property name="virtual_phone_glass_thickness" value="0.001"/>
-      <xacro:property name="virtual_phone_body_thickness"
-                      value="${virtual_phone_thickness - virtual_phone_glass_thickness}"/>
       <link name="${namespace}virtual_phone_link">
         <visual name="phone_body_visual">
-          <origin xyz="0 0 ${virtual_phone_screen_offset + virtual_phone_body_thickness / 2.0}"/>
-          <geometry><box size="${virtual_phone_width} ${virtual_phone_height} ${virtual_phone_body_thickness}"/></geometry>
+          <origin xyz="0 0 ${virtual_phone_screen_offset + virtual_phone_thickness / 2.0}"/>
+          <geometry><box size="${virtual_phone_width} ${virtual_phone_height} ${virtual_phone_thickness}"/></geometry>
           <material name="${namespace}virtual_phone_body_material"><color rgba="0.08 0.10 0.14 1"/></material>
         </visual>
-        <collision name="${namespace}virtual_phone_body_collision">
-          <origin xyz="0 0 ${virtual_phone_screen_offset + virtual_phone_body_thickness / 2.0}"/>
-          <geometry><box size="${virtual_phone_width} ${virtual_phone_height} ${virtual_phone_body_thickness}"/></geometry>
-        </collision>
       </link>
       <joint name="${namespace}virtual_phone_joint" type="fixed">
@@ -182,13 +175,8 @@
       <link name="${namespace}virtual_phone_screen_frame">
         <visual name="screen_visual">
-          <!-- This link is the physical screen plane. The OBJ/MTL preserves
-               UV mapping in both RViz and Gazebo. -->
+          <!-- The OBJ/MTL preserves UV mapping in RViz and Gazebo. -->
           <origin xyz="0 0 0.00001" rpy="0 0 0"/>
           <geometry><mesh filename="file://$(find denso_robot_descriptions)/tools/virtual_phone/meshes/phone_screen.obj" scale="${virtual_phone_height * 0.94} ${virtual_phone_height * 0.94} ${virtual_phone_height * 0.94}"/></geometry>
         </visual>
-        <collision name="${namespace}virtual_phone_screen_collision">
-          <origin xyz="0 0 ${-virtual_phone_glass_thickness / 2.0}"/>
-          <geometry><box size="${virtual_phone_width * 0.94} ${virtual_phone_height * 0.94} ${virtual_phone_glass_thickness}"/></geometry>
-        </collision>
       </link>
       <joint name="${namespace}virtual_phone_screen_joint" type="fixed">
